File: pcb/MCP23008/MCP23008.sch (KiCad schematic (older format))
At the start: 5 parts, among them U3 PCF8574

Commit message: digikey lib, mcp subproject
Parts:
- removed D1: LED, LED_SMD:LED_0603_1608Metric, symbol Device:LED
- removed R5, R7, R8: 1K, Resistor_SMD:R_0603_1608Metric, symbol Device:R
- removed U3: PCF8574, pcf8574:SO16W, symbol Interface_Expansion:PCF8574
- added J1, J2, J3: Conn_01x03_Male, symbol Connector:Conn_01x03_Male
- added J4: Conn_01x08_Male, symbol Connector:Conn_01x08_Male
- added J5: Conn_01x04_Male, symbol Connector:Conn_01x04_Male
- added R1, R2: 1K, symbol Device:R_Small
- added U1: MCP23008-E_P, digikey-footprints:DIP-18_W7.62mm, symbol dk_Interface-I-O-Expanders:MCP23008-E_P
Connections:
- net GND: now also J1.3 (Pin_3), J2.3 (Pin_3), J3.3 (Pin_3), J5.4 (Pin_4), U1.8 (INT), U1.9 (VSS)
- net SCL: now also J5.3 (Pin_3), R1.2, U1.1 (SCL)
- net SDA: now also J5.2 (Pin_2), R2.2, U1.2 (SDA)
- net VCC: now also J1.1 (Pin_1), J2.1 (Pin_1), J3.1 (Pin_1), J5.1 (Pin_1), R1.1, R2.1, U1.18 (VDD), U1.6 (~RESET)
- new net: J4.1 (Pin_1), U1.10 (GP0)
- new net: J4.2 (Pin_2), U1.11 (GP1)
- new net: J4.3 (Pin_3), U1.12 (GP2)
- new net: J4.4 (Pin_4), U1.13 (GP3)
- new net: J4.5 (Pin_5), U1.14 (GP4)
- new net: J4.6 (Pin_6), U1.15 (GP5)
- new net: J4.7 (Pin_7), U1.16 (GP6)
- new net: J4.8 (Pin_8), U1.17 (GP7)
- new net: J1.2 (Pin_2), U1.3 (A2)
- new net: J2.2 (Pin_2), U1.4 (A1)
- new net: J3.2 (Pin_2), U1.5 (A0)
- no-connect marks 1 -> 0

Commit message: make lib paths relative, add footprints to mcp23008 breakout, chuck into pcbnew
Parts:
- J1, J2, J3: footprint (none) -> Connector_PinSocket_2.54mm:PinSocket_1x03_P2.54mm_Vertical
- J4: footprint (none) -> Connector_PinSocket_2.54mm:PinSocket_1x08_P2.54mm_Vertical
- J5: footprint (none) -> Connector_PinSocket_2.54mm:PinSocket_1x04_P2.54mm_Vertical
- R1, R2: footprint (none) -> Resistor_THT:R_Axial_DIN0204_L3.6mm_D1.6mm_P2.54mm_Vertical
Changed lines of the file:
@@
 EESchema Schematic File Version 4
-EELAYER 30 0
+LIBS:MCP23008-cache
+EELAYER 29 0
 EELAYER END
 $Descr A4 11693 8268
@@
 F 0 "J1" H 2108 5381 50  0000 C CNN
 F 1 "Conn_01x03_Male" H 2108 5290 50  0000 C CNN
-F 2 "" H 2000 5100 50  0001 C CNN
+F 2 "Connector_PinSocket_2.54mm:PinSocket_1x03_P2.54mm_Vertical" H 2000 5100 50  0001 C CNN
 F 3 "~" H 2000 5100 50  0001 C CNN
 	1    2000 5100
@@
 F 0 "J2" H 2108 5831 50  0000 C CNN
 F 1 "Conn_01x03_Male" H 2108 5740 50  0000 C CNN
-F 2 "" H 2000 5550 50  0001 C CNN
+F 2 "Connector_PinSocket_2.54mm:PinSocket_1x03_P2.54mm_Vertical" H 2000 5550 50  0001 C CNN
 F 3 "~" H 2000 5550 50  0001 C CNN
 	1    2000 5550
@@
 F 0 "J3" H 2108 6281 50  0000 C CNN
 F 1 "Conn_01x03_Male" H 2108 6190 50  0000 C CNN
-F 2 "" H 2000 6000 50  0001 C CNN
+F 2 "Connector_PinSocket_2.54mm:PinSocket_1x03_P2.54mm_Vertical" H 2000 6000 50  0001 C CNN
 F 3 "~" H 2000 6000 50  0001 C CNN
 	1    2000 6000
@@
 F 0 "J4" H 3058 4681 50  0000 C CNN
 F 1 "Conn_01x08_Male" H 3058 4590 50  0000 C CNN
-F 2 "" H 2950 4200 50  0001 C CNN
+F 2 "Connector_PinSocket_2.54mm:PinSocket_1x08_P2.54mm_Vertical" H 2950 4200 50  0001 C CNN
 F 3 "~" H 2950 4200 50  0001 C CNN
 	1    2950 4200
@@
 F 0 "J5" H 1258 4481 50  0000 C CNN
 F 1 "Conn_01x04_Male" H 1258 4390 50  0000 C CNN
-F 2 "" H 1150 4200 50  0001 C CNN
+F 2 "Connector_PinSocket_2.54mm:PinSocket_1x04_P2.54mm_Vertical" H 1150 4200 50  0001 C CNN
 F 3 "~" H 1150 4200 50  0001 C CNN
 	1    1150 4200
@@
 F 0 "R1" V 2896 4850 50  0000 C CNN
 F 1 "1K" V 2805 4850 50  0000 C CNN
-F 2 "" H 2700 4850 50  0001 C CNN
+F 2 "Resistor_THT:R_Axial_DIN0204_L3.6mm_D1.6mm_P2.54mm_Vertical" H 2700 4850 50  0001 C CNN
 F 3 "~" H 2700 4850 50  0001 C CNN
 	1    2700 4850
@@
 F 0 "R2" V 2896 4550 50  0000 C CNN
 F 1 "1K" V 2805 4550 50  0000 C CNN
-F 2 "" H 2700 4550 50  0001 C CNN
+F 2 "Resistor_THT:R_Axial_DIN0204_L3.6mm_D1.6mm_P2.54mm_Vertical" H 2700 4550 50  0001 C CNN
 F 3 "~" H 2700 4550 50  0001 C CNN
 	1    2700 4550
