File: pcb/MCP23008/MCP23008.kicad_pcb (KiCad board)
At the start: 2 copper layers, 8 parts, among them J1 Conn_01x03_Male, J2 Conn_01x03_Male, J3 Conn_01x03_Male, J4 Conn_01x08_Male, J5 Conn_01x04_Male, U1 MCP23008-E_P

Commit message: frame
Parts:
- J1: value Conn_01x03_Male -> A0
- J2: value Conn_01x03_Male -> A1
- J3: value Conn_01x03_Male -> A2
- J4: value Conn_01x08_Male -> IO
- J5: value Conn_01x04_Male -> Input
- moved J1 22.6 mm to (99.1, 115.6), turned to 90 degrees
- moved R1 18.0 mm to (104.1, 108.0), turned to 270 degrees
- moved J5 15.9 mm to (100.3, 101.6)
- moved J2 13.4 mm to (99.1, 118.1), turned to 90 degrees
- moved R2 12.5 mm to (104.1, 102.9), turned to 90 degrees
- moved J4 11.3 mm to (119.4, 120.7)
- moved J3 5.26 mm to (99.1, 120.7), turned to 90 degrees
- moved U1 1.67 mm to (108.0, 100.3)
Other:
- board outline added: 27.9 x 26.7 mm
- board text added: "GND"
- board text added: "SCL"
- board text added: "SDA"
- board text added: "VCC"
