File: pcb/MCP23008/MCP23008.kicad_pcb (KiCad board)
At the start: 2 copper layers, 27.9 x 26.7 mm, 8 parts, among them J1 A0, J2 A1, J3 A2, J4 IO, J5 Input, U1 MCP23008-E_P

Commit message: route mcp23008
Routing:
- net VCC: track 0.00 -> 43.7 mm
- net GND: track 0.00 -> 19.4 mm
- net /SCL: track 0.00 -> 16.9 mm
- net Net-(J3-Pad2): track 0.00 -> 13.1 mm
- net Net-(J2-Pad2): track 0.00 -> 12.9 mm
- net Net-(J1-Pad2): track 0.00 -> 12.8 mm
- net /SDA: track 0.00 -> 10.9 mm
- net Net-(J4-Pad8): track 0.00 -> 3.81 mm
- net Net-(J4-Pad7): track 0.00 -> 3.81 mm
- net Net-(J4-Pad6): track 0.00 -> 3.81 mm
- net Net-(J4-Pad5): track 0.00 -> 3.81 mm
- net Net-(J4-Pad4): track 0.00 -> 3.81 mm
- net Net-(J4-Pad3): track 0.00 -> 3.81 mm
- net Net-(J4-Pad2): track 0.00 -> 3.81 mm
- net Net-(J4-Pad1): track 0.00 -> 3.81 mm
Other:
- net class Default: clearance 0.2 -> 0.1524; trace_width 0.25 -> 0.1524; via_dia 0.8 -> 0.508; via_drill 0.4 -> 0.254
- rule pad_to_mask_clearance: 0 -> 0.0508
- rule trace_clearance: 0.2 -> 0.1524
- rule trace_min: 0.2 -> 0.1524
- rule via_min_drill: 0.3 -> 0.254
- rule via_min_size: 0.4 -> 0.508
Changed lines of the file:
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@@
-(kicad_pcb (version 20171130) (host pcbnew 5.1.5-52549c5~86~ubuntu18.04.1)
+(kicad_pcb (version 20171130) (host pcbnew "(5.1.2)-1")
   (general
     (thickness 1.6)
     (drawings 8)
-    (tracks 0)
+    (tracks 62)
     (zones 0)
     (modules 8)
@@
   )
   (setup
-    (last_trace_width 0.25)
-    (trace_clearance 0.2)
+    (last_trace_width 0.1524)
+    (user_trace_width 0.1524)
+    (user_trace_width 0.508)
+    (trace_clearance 0.1524)
     (zone_clearance 0.508)
     (zone_45_only no)
-    (trace_min 0.2)
-    (via_size 0.8)
-    (via_drill 0.4)
-    (via_min_size 0.4)
-    (via_min_drill 0.3)
-    (uvia_size 0.3)
-    (uvia_drill 0.1)
+    (trace_min 0.1524)
+    (via_size 0.508)
+    (via_drill 0.254)
+    (via_min_size 0.508)
+    (via_min_drill 0.254)
+    (uvia_size 0.508)
+    (uvia_drill 0.254)
     (uvias_allowed no)
-    (uvia_min_size 0.2)
-    (uvia_min_drill 0.1)
+    (uvia_min_size 0.508)
+    (uvia_min_drill 0.254)
     (edge_width 0.1)
     (segment_width 0.2)
@@
     (pad_size 1.524 1.524)
     (pad_drill 0.762)
-    (pad_to_mask_clearance 0)
+    (pad_to_mask_clearance 0.0508)
+    (solder_mask_min_width 0.0508)
     (aux_axis_origin 0 0)
-    (visible_elements FFFFF77F)
+    (visible_elements 7FFFFFFF)
     (pcbplotparams
       (layerselection 0x010fc_ffffffff)
@@
   (net 16 "Net-(U1-Pad7)")
   (net_class Default "This is the default net class."
-    (clearance 0.2)
-    (trace_width 0.25)
-    (via_dia 0.8)
-    (via_drill 0.4)
-    (uvia_dia 0.3)
-    (uvia_drill 0.1)
+    (clearance 0.1524)
+    (trace_width 0.1524)
+    (via_dia 0.508)
+    (via_drill 0.254)
+    (uvia_dia 0.508)
+    (uvia_drill 0.254)
     (add_net /SCL)
     (add_net /SDA)
@@
     (effects (font (size 1 1) (thickness 0.15)))
   )
+  (segment (start 107.95 118.11) (end 107.95 120.65) (width 0.1524) (layer B.Cu) (net 1))
+  (segment (start 100.33 109.22) (end 100.33 110.2989) (width 0.1524) (layer F.Cu) (net 1))
+  (segment (start 100.33 110.2989) (end 104.14 114.1089) (width 0.1524) (layer F.Cu) (net 1))
+  (segment (start 104.14 114.1089) (end 104.14 115.57) (width 0.1524) (layer F.Cu) (net 1))
+  (segment (start 104.14 118.11) (end 107.95 118.11) (width 0.1524) (layer F.Cu) (net 1))
+  (segment (start 104.14 118.11) (end 104.14 120.65) (width 0.1524) (layer B.Cu) (net 1))
+  (segment (start 104.14 115.57) (end 104.14 118.11) (width 0.1524) (layer B.Cu) (net 1))
+  (segment (start 101.6 115.57) (end 101.6 114.4911) (width 0.1524) (layer B.Cu) (net 2))
+  (segment (start 101.6 114.4911) (end 106.439 109.6521) (width 0.1524) (layer B.Cu) (net 2))
+  (segment (start 106.439 109.6521) (end 106.439 106.921) (width 0.1524) (layer B.Cu) (net 2))
+  (segment (start 106.439 106.921) (end 107.95 105.41) (width 0.1524) (layer B.Cu) (net 2))
+  (segment (start 104.7827 107.95) (end 104.7827 104.2911) (width 0.1524) (layer F.Cu) (net 3))
+  (segment (start 104.7827 104.2911) (end 105.1719 103.9019) (width 0.1524) (layer F.Cu) (net 3))
+  (segment (start 107.95 113.03) (end 106.439 111.519) (width 0.1524) (layer F.Cu) (net 3))
+  (segment (start 106.439 111.519) (end 106.439 109.6063) (width 0.1524) (layer F.Cu) (net 3))
+  (segment (start 106.439 109.6063) (end 104.7827 107.95) (width 0.1524) (layer F.Cu) (net 3))
+  (segment (start 104.14 107.95) (end 104.7827 107.95) (width 0.1524) (layer F.Cu) (net 3))
+  (segment (start 105.1719 103.9019) (end 104.14 102.87) (width 0.1524) (layer F.Cu) (net 3))
+  (segment (start 115.57 100.33) (end 111.9981 103.9019) (width 0.1524) (layer F.Cu) (net 3))
+  (segment (start 111.9981 103.9019) (end 105.1719 103.9019) (width 0.1524) (layer F.Cu) (net 3))
+  (segment (start 104.14 102.87) (end 102.6789 102.87) (width 0.1524) (layer F.Cu) (net 3))
+  (segment (start 102.6789 102.87) (end 101.4089 101.6) (width 0.1524) (layer F.Cu) (net 3))
+  (segment (start 100.33 101.6) (end 101.4089 101.6) (width 0.1524) (layer F.Cu) (net 3))
+  (segment (start 104.14 107.95) (end 99.06 113.03) (width 0.1524) (layer B.Cu) (net 3))
+  (segment (start 99.06 113.03) (end 99.06 114.4911) (width 0.1524) (layer B.Cu) (net 3))
+  (segment (start 99.06 115.57) (end 99.06 114.4911) (width 0.1524) (layer B.Cu) (net 3))
+  (segment (start 99.06 118.11) (end 99.06 120.65) (width 0.1524) (layer B.Cu) (net 3))
+  (segment (start 99.06 115.57) (end 99.06 118.11) (width 0.1524) (layer B.Cu) (net 3))
+  (segment (start 101.6 118.11) (end 101.6 117.0311) (width 0.1524) (layer B.Cu) (net 4))
+  (segment (start 101.6 117.0311) (end 101.735 117.0311) (width 0.1524) (layer B.Cu) (net 4))
+  (segment (start 101.735 117.0311) (end 102.6789 116.0872) (width 0.1524) (layer B.Cu) (net 4))
+  (segment (start 102.6789 116.0872) (end 102.6789 114.3059) (width 0.1524) (layer B.Cu) (net 4))
+  (segment (start 102.6789 114.3059) (end 107.95 109.0348) (width 0.1524) (layer B.Cu) (net 4))
+  (segment (start 107.95 109.0348) (end 107.95 107.95) (width 0.1524) (layer B.Cu) (net 4))
+  (segment (start 101.6 120.65) (end 101.6 119.5711) (width 0.1524) (layer B.Cu) (net 5))
+  (segment (start 101.6 119.5711) (end 101.7349 119.5711) (width 0.1524) (layer B.Cu) (net 5))
+  (segment (start 101.7349 119.5711) (end 102.9841 118.3219) (width 0.1524) (layer B.Cu) (net 5))
+  (segment (start 102.9841 118.3219) (end 102.9841 115.1155) (width 0.1524) (layer B.Cu) (net 5))
+  (segment (start 102.9841 115.1155) (end 107.6096 110.49) (width 0.1524) (layer B.Cu) (net 5))
+  (segment (start 107.6096 110.49) (end 107.95 110.49) (width 0.1524) (layer B.Cu) (net 5))
+  (segment (start 119.38 102.87) (end 115.57 102.87) (width 0.1524) (layer F.Cu) (net 6))
+  (segment (start 119.38 105.41) (end 115.57 105.41) (width 0.1524) (layer F.Cu) (net 7))
+  (segment (start 119.38 107.95) (end 115.57 107.95) (width 0.1524) (layer F.Cu) (net 8))
+  (segment (start 119.38 110.49) (end 115.57 110.49) (width 0.1524) (layer F.Cu) (net 9))
+  (segment (start 119.38 113.03) (end 115.57 113.03) (width 0.1524) (layer F.Cu) (net 10))
+  (segment (start 119.38 115.57) (end 115.57 115.57) (width 0.1524) (layer F.Cu) (net 11))
+  (segment (start 119.38 118.11) (end 115.57 118.11) (width 0.1524) (layer F.Cu) (net 12))
+  (segment (start 119.38 120.65) (end 115.57 120.65) (width 0.1524) (layer F.Cu) (net 13))
+  (segment (start 107.95 100.33) (end 107.95 101.3589) (width 0.1524) (layer B.Cu) (net 14))
+  (segment (start 100.33 106.68) (end 102.6289 106.68) (width 0.1524) (layer B.Cu) (net 14))
+  (segment (start 102.6289 106.68) (end 107.95 101.3589) (width 0.1524) (layer B.Cu) (net 14))
+  (segment (start 104.14 110.49) (end 104.14 109.5611) (width 0.1524) (layer F.Cu) (net 14))
+  (segment (start 100.33 106.68) (end 101.4089 106.68) (width 0.1524) (layer F.Cu) (net 14))
+  (segment (start 101.4089 106.68) (end 101.4089 106.83) (width 0.1524) (layer F.Cu) (net 14))
+  (segment (start 101.4089 106.83) (end 104.14 109.5611) (width 0.1524) (layer F.Cu) (net 14))
+  (segment (start 104.14 100.33) (end 105.0689 100.33) (width 0.1524) (layer F.Cu) (net 15))
+  (segment (start 105.0689 100.33) (end 107.6089 102.87) (width 0.1524) (layer F.Cu) (net 15))
+  (segment (start 107.6089 102.87) (end 107.95 102.87) (width 0.1524) (layer F.Cu) (net 15))
+  (segment (start 104.14 100.33) (end 104.14 101.2589) (width 0.1524) (layer B.Cu) (net 15))
+  (segment (start 100.33 104.14) (end 101.4089 104.14) (width 0.1524) (layer B.Cu) (net 15))
+  (segment (start 101.4089 104.14) (end 101.4089 103.99) (width 0.1524) (layer B.Cu) (net 15))
+  (segment (start 101.4089 103.99) (end 104.14 101.2589) (width 0.1524) (layer B.Cu) (net 15))
 )
