File: pcb/avr-gamepad.sch (KiCad schematic (older format))
At the start: 56 parts, among them J1 Conn_01x06, J2 Conn_01x06, J3 Conn_01x05, J4 Conn_01x05, P1 USB_C_Plug_USB2.0, SW1 RESET, SW10 R2, SW11 A, SW13 Left, SW14 L2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

Commit message: change triggers to tact switches, add footprint
Parts:
- SW10, SW14, SW8: footprint button-contacts:Small -> right-angle-tact:TL3330
- SW7: footprint button-contacts:Large_tapered -> right-angle-tact:TL3330
Changed lines of the file:
@@
 F 0 "SW14" H 8450 2185 50  0000 C CNN
 F 1 "L2" H 8450 2094 50  0000 C CNN
-F 2 "button-contacts:Small" H 8450 2100 50  0001 C CNN
+F 2 "right-angle-tact:TL3330" H 8450 2100 50  0001 C CNN
 F 3 "~" H 8450 2100 50  0001 C CNN
 	1    8450 1900
@@
 F 0 "SW7" H 8450 1185 50  0000 C CNN
 F 1 "L1" H 8450 1094 50  0000 C CNN
-F 2 "button-contacts:Large_tapered" H 8450 1100 50  0001 C CNN
+F 2 "right-angle-tact:TL3330" H 8450 1100 50  0001 C CNN
 F 3 "~" H 8450 1100 50  0001 C CNN
 	1    8450 900
@@
 F 0 "SW8" H 5100 1685 50  0000 C CNN
 F 1 "R1" H 5100 1594 50  0000 C CNN
-F 2 "button-contacts:Small" H 5100 1600 50  0001 C CNN
+F 2 "right-angle-tact:TL3330" H 5100 1600 50  0001 C CNN
 F 3 "~" H 5100 1600 50  0001 C CNN
 	1    5100 1400
@@
 F 0 "SW10" H 5100 2185 50  0000 C CNN
 F 1 "R2" H 5100 2094 50  0000 C CNN
-F 2 "button-contacts:Small" H 5100 2100 50  0001 C CNN
+F 2 "right-angle-tact:TL3330" H 5100 2100 50  0001 C CNN
 F 3 "~" H 5100 2100 50  0001 C CNN
 	1    5100 1900

Commit message: change 5-pin ffc to molex
Parts:
- J3, J4: footprint uxcell-ffc:uxcell_ffc_0.5pitch_1x05 -> molex_5051100592:5051100592
Changed lines of the file:
@@
 F 0 "J3" H 5292 3235 50  0000 C CNN
 F 1 "Conn_01x05" H 5292 3144 50  0000 C CNN
-F 2 "uxcell-ffc:uxcell_ffc_0.5pitch_1x05" H 5400 2750 50  0001 C CNN
+F 2 "molex_5051100592:5051100592" H 5400 2750 50  0001 C CNN
 F 3 "~" H 5400 2750 50  0001 C CNN
 	1    5400 2750
@@
 F 0 "J4" H 10592 3285 50  0000 C CNN
 F 1 "Conn_01x05" H 10592 3194 50  0000 C CNN
-F 2 "uxcell-ffc:uxcell_ffc_0.5pitch_1x05" H 10700 2800 50  0001 C CNN
+F 2 "molex_5051100592:5051100592" H 10700 2800 50  0001 C CNN
 F 3 "~" H 10700 2800 50  0001 C CNN
 	1    10700 2800

Commit message: improve d-pad contacts
Parts:
- SW13, SW2, SW3, SW4: footprint button-contacts:Large_tapered -> button-contacts:Dpad_Large_tapered
Changed lines of the file:
@@
 F 0 "SW3" H 9300 1185 50  0000 C CNN
 F 1 "Up" H 9300 1094 50  0000 C CNN
-F 2 "button-contacts:Large_tapered" H 9300 1100 50  0001 C CNN
+F 2 "button-contacts:Dpad_Large_tapered" H 9300 1100 50  0001 C CNN
 F 3 "~" H 9300 1100 50  0001 C CNN
 	1    9300 900
@@
 F 0 "SW4" H 9300 1685 50  0000 C CNN
 F 1 "Down" H 9300 1594 50  0000 C CNN
-F 2 "button-contacts:Large_tapered" H 9300 1600 50  0001 C CNN
+F 2 "button-contacts:Dpad_Large_tapered" H 9300 1600 50  0001 C CNN
 F 3 "~" H 9300 1600 50  0001 C CNN
 	1    9300 1400
@@
 F 0 "SW2" H 10150 1685 50  0000 C CNN
 F 1 "Right" H 10150 1594 50  0000 C CNN
-F 2 "button-contacts:Large_tapered" H 10150 1600 50  0001 C CNN
+F 2 "button-contacts:Dpad_Large_tapered" H 10150 1600 50  0001 C CNN
 F 3 "~" H 10150 1600 50  0001 C CNN
 	1    10150 1400
@@
 F 0 "SW13" H 8450 1685 50  0000 C CNN
 F 1 "Left" H 8450 1594 50  0000 C CNN
-F 2 "button-contacts:Large_tapered" H 8450 1600 50  0001 C CNN
+F 2 "button-contacts:Dpad_Large_tapered" H 8450 1600 50  0001 C CNN
 F 3 "~" H 8450 1600 50  0001 C CNN
 	1    8450 1400
